File: easyeda/DECA_ALU_EasyEDA_Schematic.sch (EAGLE design)
At the start: 36 parts, among them IC1 4-Bit Binary Full Adder, IC10 Bit 3 8:1 MUX, IC11 Commercial 4-Bit ALU, IC12 4-Bit Magnitude Comparator, IC2 Subtraction Invert XOR, IC3 Bitwise XOR Array, IC4 Bitwise AND Array, IC5 Bitwise OR Array, IC6 Hex Inverter Array, IC7 Bit 0 8:1 MUX, IC8 Bit 1 8:1 MUX, IC9 Bit 2 8:1 MUX

Commit message: fix(easyeda): scale schematic grid to standard millimeters for clean EasyEDA layout
Parts:
- removed R_BOT0, R_BOT1, R_BOT2, R_BOT3, R_BOT4, R_BOT5, R_BOT6, R_BOT7, R_BOT8: 4.7kΩ (Divider Bottom), DECA_ALU_LIB:RESISTOR
- removed R_TOP0, R_TOP1, R_TOP2, R_TOP3, R_TOP4, R_TOP5, R_TOP6, R_TOP7, R_TOP8: 2.2kΩ (Divider Top), DECA_ALU_LIB:RESISTOR
Connections:
- net SILICON_MATCH: no longer R_TOP8.1
- net Y0_BUS: no longer R_TOP0.1
- net Y1_BUS: no longer R_TOP1.1
- net Y2_BUS: no longer R_TOP2.1
- net Y3_BUS: no longer R_TOP3.1
